File: hardware/kicad/temperature_logger/001_Power.sch (KiCad schematic (older format))
At the start: 22 parts, among them J2 Power, J3 USB_B_Micro, Q1 Q_PMOS_DGS, U4 AMS1117-3.3, U5 FT231XS

Commit message: Hardware routing completed (verification required)
Parts:
- removed Q1: Q_PMOS_DGS, Package_TO_SOT_SMD:SOT-23, symbol Device:Q_PMOS_DGS
- added Q1: Q_PMOS_GSD, Package_TO_SOT_SMD:SOT-23, symbol Device:Q_PMOS_GSD
Changed lines of the file:
@@
 	5500 1300 5500 1400
-Wire Wire Line
-	6100 1300 6450 1300
 Wire Wire Line
 	6450 1300 6450 1200
@@
 Wire Wire Line
 	5500 2750 5500 2850
-$Comp
-L Device:Q_PMOS_DGS Q?
-U 1 1 60D6C346
-P 5400 1600
-AR Path="/60D6C346" Ref="Q?"  Part="1"
-AR Path="/60D5E44C/60D6C346" Ref="Q1"  Part="1"
-F 0 "Q1" H 5605 1554 50  0000 L CNN
-F 1 "Q_PMOS_DGS" H 5605 1645 50  0000 L CNN
-F 2 "Package_TO_SOT_SMD:SOT-23" H 5600 1700 50  0001 C CNN
-F 3 "~" H 5400 1600 50  0001 C CNN
-	1    5400 1600
-	1    0    0    1
-$EndComp
 Wire Wire Line
 	5500 2550 5500 2450
@@
 Wire Wire Line
 	6500 3000 6500 2900
+$Comp
+L Device:Q_PMOS_GSD Q1
+U 1 1 60D8512E
+P 5400 1600
+F 0 "Q1" H 5605 1554 50  0000 L CNN
+F 1 "Q_PMOS_GSD" H 5605 1645 50  0000 L CNN
+F 2 "Package_TO_SOT_SMD:SOT-23" H 5600 1700 50  0001 C CNN
+F 3 "~" H 5400 1600 50  0001 C CNN
+	1    5400 1600
+	1    0    0    1
+$EndComp
+Wire Wire Line
+	6100 1300 6450 1300
 $EndSCHEMATC
