File: hardware/kicad/temperature_logger/temperature_logger.sch (KiCad schematic (older format))
At the start: 23 parts, among them J1 SWD, J4 UART, SW1 UserBtn, U1 TMP112, U2 MX25R1635FM1IL0, U3 STM32L053C8Tx

Commit message: Main rounting done for pass 2
Parts:
- J1: footprint Connector_PinHeader_1.27mm:PinHeader_1x06_P1.27mm_Vertical -> Connector_PinHeader_1.27mm:PinHeader_1x05_P1.27mm_Vertical
Connections:
- net TMP_ALERT: now also U3.42 (PB6); no longer U3.18 (PB0)
- net USER_BTN: now also U3.33 (PA12); no longer U3.10 (PA0)
- net USER_LED1: now also U3.40 (PB4); no longer U3.15 (PA5)
- net USER_LED2: now also U3.39 (PB3); no longer U3.40 (PB4)
Changed lines of the file:
@@
 Wire Wire Line
 	8500 3600 8000 3600
-Wire Wire Line
-	9700 3700 10250 3700
 Text Label 8000 3600 0    50   ~ 0
-USER_LED2
-Text Label 10250 3700 2    50   ~ 0
 USER_LED1
 Wire Wire Line
-	9700 3200 10250 3200
-Text Label 10250 3200 2    50   ~ 0
+	9700 4400 10250 4400
+Text Label 10250 4400 2    50   ~ 0
 USER_BTN
 Wire Wire Line
@@
 FLASH_RSTN
 Wire Wire Line
-	8500 3200 8000 3200
-Text Label 8000 3200 0    50   ~ 0
+	8500 3800 8000 3800
+Text Label 8000 3800 0    50   ~ 0
 TMP_ALERT
 Wire Wire Line
@@
 Text Label 10250 4600 2    50   ~ 0
 SWCLK
-NoConn ~ 8500 3500
 NoConn ~ 8500 3700
-NoConn ~ 8500 3800
 NoConn ~ 8500 3900
 NoConn ~ 8500 4200
 NoConn ~ 8500 4300
 NoConn ~ 9700 4700
-NoConn ~ 9700 4400
 NoConn ~ 9700 4300
 NoConn ~ 9700 4000
@@
 F 0 "J1" H 1358 7631 50  0000 C CNN
 F 1 "SWD" H 1358 7540 50  0000 C CNN
-F 2 "Connector_PinHeader_1.27mm:PinHeader_1x06_P1.27mm_Vertical" H 1250 7250 50  0001 C CNN
+F 2 "Connector_PinHeader_1.27mm:PinHeader_1x05_P1.27mm_Vertical" H 1250 7250 50  0001 C CNN
 F 3 "~" H 1250 7250 50  0001 C CNN
 	1    1250 7250
@@
 Wire Wire Line
 	3050 7250 3050 7300
+Text Label 8000 3500 0    50   ~ 0
+USER_LED2
+NoConn ~ 9700 3700
+Wire Wire Line
+	8500 3500 8000 3500
+NoConn ~ 9700 3200
+NoConn ~ 8500 3200
 $EndSCHEMATC

Commit message: Hardware routing completed (verification required)
Parts:
- removed SW1: UserBtn, Button_Switch_SMD:SW_SPST_Omron_B3FS-101xP, symbol Switch:SW_Push
- added SW1: SW_MEC_5E, Button_Switch_SMD:SW_SPST_Omron_B3FS-101xP, symbol Switch:SW_MEC_5E
- J1: footprint Connector_PinHeader_1.27mm:PinHeader_1x05_P1.27mm_Vertical -> Connector_PinHeader_2.54mm:PinHeader_1x05_P2.54mm_Vertical
- J4: footprint Connector_PinHeader_1.27mm:PinHeader_1x03_P1.27mm_Vertical -> Connector_PinHeader_2.54mm:PinHeader_1x03_P2.54mm_Vertical
Connections:
- wire segments 122 -> 126
Changed lines of the file:
@@
 USER_LED1
-$Comp
-L Switch:SW_Push SW1
-U 1 1 60C6A850
-P 2800 5500
-F 0 "SW1" V 2754 5648 50  0000 L CNN
-F 1 "UserBtn" V 2845 5648 50  0000 L CNN
-F 2 "Button_Switch_SMD:SW_SPST_Omron_B3FS-101xP" H 2800 5700 50  0001 C CNN
-F 3 "~" H 2800 5700 50  0001 C CNN
-	1    2800 5500
-	0    1    1    0
-$EndComp
 $Comp
 L power:GND #PWR010
@@
 	1    0    0    -1
 $EndComp
-Wire Wire Line
-	2800 5700 2800 5750
-Wire Wire Line
-	2800 5250 2800 5300
 $Comp
 L Device:C_Small C2
@@
 F 3 "" H 2850 3600 50  0001 C CNN
 	1    2850 3600
-	1    0    0    -1
-$EndComp
-$Comp
-L power:VDC #PWR09
-U 1 1 60CD3BDE
-P 2800 5250
-F 0 "#PWR09" H 2800 5150 50  0001 C CNN
-F 1 "VDC" H 2815 5423 50  0000 C CNN
-F 2 "" H 2800 5250 50  0001 C CNN
-F 3 "" H 2800 5250 50  0001 C CNN
-	1    2800 5250
 	1    0    0    -1
 $EndComp
@@
 F 0 "J1" H 1358 7631 50  0000 C CNN
 F 1 "SWD" H 1358 7540 50  0000 C CNN
-F 2 "Connector_PinHeader_1.27mm:PinHeader_1x05_P1.27mm_Vertical" H 1250 7250 50  0001 C CNN
+F 2 "Connector_PinHeader_2.54mm:PinHeader_1x05_P2.54mm_Vertical" H 1250 7250 50  0001 C CNN
 F 3 "~" H 1250 7250 50  0001 C CNN
 	1    1250 7250
@@
 F 0 "J4" H 2758 7431 50  0000 C CNN
 F 1 "UART" H 2758 7340 50  0000 C CNN
-F 2 "Connector_PinHeader_1.27mm:PinHeader_1x03_P1.27mm_Vertical" H 2650 7150 50  0001 C CNN
+F 2 "Connector_PinHeader_2.54mm:PinHeader_1x03_P2.54mm_Vertical" H 2650 7150 50  0001 C CNN
 F 3 "~" H 2650 7150 50  0001 C CNN
 	1    2650 7150
@@
 NoConn ~ 9700 3200
 NoConn ~ 8500 3200
+$Comp
+L Switch:SW_MEC_5E SW1
+U 1 1 60D808BB
+P 2850 5300
+F 0 "SW1" V 2896 5212 50  0000 R CNN
+F 1 "SW_MEC_5E" V 2805 5212 50  0000 R CNN
+F 2 "Button_Switch_SMD:SW_SPST_Omron_B3FS-101xP" H 2850 5600 50  0001 C CNN
+F 3 "http://www.apem.com/int/index.php?controller=attachment&id_attachment=1371" H 2850 5600 50  0001 C CNN
+	1    2850 5300
+	0    -1   -1   0
+$EndComp
+Wire Wire Line
+	2750 5500 2800 5500
+Wire Wire Line
+	2750 5100 2800 5100
+$Comp
+L power:VDC #PWR09
+U 1 1 60D9A862
+P 2800 4950
+F 0 "#PWR09" H 2800 4850 50  0001 C CNN
+F 1 "VDC" H 2815 5123 50  0000 C CNN
+F 2 "" H 2800 4950 50  0001 C CNN
+F 3 "" H 2800 4950 50  0001 C CNN
+	1    2800 4950
+	1    0    0    -1
+$EndComp
+Wire Wire Line
+	2800 4950 2800 5100
+Connection ~ 2800 5100
+Wire Wire Line
+	2800 5100 2850 5100
+Wire Wire Line
+	2800 5500 2800 5750
+Connection ~ 2800 5500
+Wire Wire Line
+	2800 5500 2850 5500
 $EndSCHEMATC

Commit message: Added schematic changes
Other:
- note added: "Microcontroller"
- moved on the sheet: R8
Changed lines of the file:
@@
 encoding utf-8
 Sheet 1 2
-Title ""
-Date ""
-Rev ""
-Comp ""
+Title "Temperature Logger"
+Date "2021-09-12"
+Rev "1"
+Comp "PradS"
 Comment1 ""
 Comment2 ""
@@
 L Device:R_Small R8
 U 1 1 60CFBBE0
-P 6950 2200
-F 0 "R8" H 7009 2246 50  0000 L CNN
-F 1 "1k" H 7009 2155 50  0000 L CNN
-F 2 "Resistor_SMD:R_0603_1608Metric_Pad1.05x0.95mm_HandSolder" H 6950 2200 50  0001 C CNN
-F 3 "~" H 6950 2200 50  0001 C CNN
-	1    6950 2200
+P 10100 2600
+F 0 "R8" H 10159 2646 50  0000 L CNN
+F 1 "1k" H 10159 2555 50  0000 L CNN
+F 2 "Resistor_SMD:R_0603_1608Metric_Pad1.05x0.95mm_HandSolder" H 10100 2600 50  0001 C CNN
+F 3 "~" H 10100 2600 50  0001 C CNN
+	1    10100 2600
 	1    0    0    -1
 $EndComp
@@
 BOOT0
 Wire Wire Line
-	6950 2100 6950 1900
-Wire Wire Line
-	6950 1900 7500 1900
+	10100 2500 10100 2300
+Wire Wire Line
+	10100 2300 10650 2300
 $Comp
 L power:GND #PWR?
 U 1 1 60D0521D
-P 6950 2450
+P 10100 2850
 AR Path="/60E10242/60D0521D" Ref="#PWR?"  Part="1"
 AR Path="/60D0521D" Ref="#PWR011"  Part="1"
-F 0 "#PWR011" H 6950 2200 50  0001 C CNN
-F 1 "GND" H 6955 2277 50  0000 C CNN
-F 2 "" H 6950 2450 50  0001 C CNN
-F 3 "" H 6950 2450 50  0001 C CNN
-	1    6950 2450
-	1    0    0    -1
-$EndComp
-Wire Wire Line
-	6950 2300 6950 2450
-Text Label 7500 1900 2    50   ~ 0
+F 0 "#PWR011" H 10100 2600 50  0001 C CNN
+F 1 "GND" H 10105 2677 50  0000 C CNN
+F 2 "" H 10100 2850 50  0001 C CNN
+F 3 "" H 10100 2850 50  0001 C CNN
+	1    10100 2850
+	1    0    0    -1
+$EndComp
+Wire Wire Line
+	10100 2700 10100 2850
+Text Label 10650 2300 2    50   ~ 0
 BOOT0
 Wire Wire Line
@@
 Wire Wire Line
 	2800 5500 2850 5500
+Wire Notes Line
+	11150 700  7600 700
+Wire Notes Line
+	7600 700  7600 5750
+Wire Notes Line
+	7600 5750 11150 5750
+Wire Notes Line
+	11150 5750 11150 700
+Text Notes 7850 5550 0    50   ~ 10
+Microcontroller
 $EndSCHEMATC
